Commit message: Moved COM of links to actual COM of links

File: ros2_ws/src/pendulum_control/urdf/macros/inertia_macros.xacro (robot description, xacro)
@@ -5,5 +5,5 @@
       <mass value="${mass}"/>
       <!-- COM at geometric center -->
-      <origin xyz="0 0 0" rpy="0 0 0"/>
+      <origin xyz="${length/2} 0 0" rpy="0 0 0"/>
       <inertia
         ixx="${(1/12.0)*mass*length*length + 0.25*mass*radius*radius}"

File: ros2_ws/src/pendulum_control/urdf/qube_constants.xacro (robot description, xacro)
@@ -8,10 +8,10 @@
   <xacro:property name="rotor_length" value="0.085"/>
   <xacro:property name="rotor_mass" value="0.095"/>
-  <xacro:property name="rotor_friction" value="0.01"/>
-  <xacro:property name="rotor_damping" value="0.05"/>
+  <xacro:property name="rotor_friction" value="0"/>
+  <xacro:property name="rotor_damping" value="0"/>
   <xacro:property name="pendulum_radius" value="0.005"/>
   <xacro:property name="pendulum_length" value="0.129"/>
   <xacro:property name="pendulum_mass" value="0.024"/>
   <xacro:property name="pendulum_friction" value="0"/>
-  <xacro:property name="pendulum_damping" value="0"/>
+  <xacro:property name="pendulum_damping" value="0.0001"/>
 </xacro:constants>
