Commit message: Added mesh to urdf file

File: ros2_ws/src/pendulum_control/urdf/joints/rotor_joint.xacro (robot description, xacro)
@@ -5,5 +5,5 @@
       <parent link="base_link"/>
       <child link="rotor_link"/>
-      <origin xyz="0 0 ${base_height+rotor_radius}" rpy="0 0 0"/>
+      <origin xyz="0 0 ${base_height+rotor_height+pendulum_height}" rpy="0 0 0"/>
       <axis xyz="0 0 1"/>
       <limit effort="2" velocity="20" lower="-1.5708" upper="1.5708"/>

File: ros2_ws/src/pendulum_control/urdf/links/base_link.xacro (robot description, xacro)
@@ -1,22 +1,30 @@
 <?xml version="1.0"?>
 <robot xmlns:xacro="http://www.ros.org/wiki/xacro" name="link_macros">
-  <xacro:macro name="base_link" params="base_width base_depth base_height base_mass">
+  <xacro:macro name="base_link" params="">
     <link name="base_link">
       <!-- Visual -->
       <visual>
-        <origin xyz="0 0 ${base_height/2}" rpy="0 0 0"/>
+        <origin xyz="0 0 0" rpy="0 0 0"/>
         <geometry>
-          <box size="${base_depth} ${base_width} ${base_height}"/>
+          <mesh filename="package://pendulum_control/urdf/mesh/base.stl" scale="0.001 0.001 0.001"/>
         </geometry>
+        <material name="green">
+          <color rgba="0 1 0 0.8"/>
+        </material>
       </visual>
       <!-- Collision -->
       <collision>
-        <origin xyz="0 0 ${base_height/2}" rpy="0 0 0"/>
+        <origin xyz="0 0 0" rpy="0 0 0"/>
         <geometry>
-          <box size="${base_width} ${base_depth} ${base_height}"/>
+          <mesh filename="package://pendulum_control/urdf/mesh/base.stl" scale="0.001 0.001 0.001"/>
         </geometry>
       </collision>
       <!-- Inertia -->
-      <xacro:base_inertia mass="${base_mass}"/>
+      <xacro:base_inertia
+        mass="${base_mass}"
+        depth="${base_depth}"
+        width="${base_width}"
+        height="${base_height}"
+      />
     </link>
   </xacro:macro>

File: ros2_ws/src/pendulum_control/urdf/links/pendulum_link.xacro (robot description, xacro)
@@ -1,34 +1,31 @@
 <?xml version="1.0"?>
 <robot xmlns:xacro="http://www.ros.org/wiki/xacro" name="link_macros">
-  <xacro:macro name="pendulum_link" params="pendulum_radius pendulum_length pendulum_mass">
+  <xacro:macro name="pendulum_link" params="">
     <link name="pendulum_link">
       <!-- Visual -->
       <visual>
-        <origin xyz="0 0 ${rotor_length/2}" rpy="0 0 0"/>
+        <origin xyz="0 0 0" rpy="0 -1.5708 0"/>
         <geometry>
-          <cylinder radius="${rotor_radius}" length="${rotor_length}"/>
-        </geometry>
-        <material name="green">
-          <color rgba="0 1 0 0.8"/>
-        </material>
-      </visual>
-      <visual>
-        <origin xyz="${pendulum_length/2-p_end_to_link-rotor_radius} 0 ${rotor_length-pendulum_radius/2}" rpy="0 1.5708 0"/>
-        <geometry>
-          <cylinder radius="${pendulum_radius}" length="${pendulum_length}"/>
+          <mesh filename="package://pendulum_control/urdf/mesh/pendulum.stl" scale="0.001 0.001 0.001"/>
         </geometry>
         <material name="orange">
-          <color rbga="1 0.65 0 0.8"/>
+          <color rgba="1 0.65 0 0.8"/>
         </material>
       </visual>
       <!-- Collision -->
       <collision>
-        <origin xyz="0 0 0" rpy="0 0 0"/>
+        <origin xyz="0 0 0" rpy="0 -1.5708 0"/>
         <geometry>
-          <cylinder radius="${pendulum_radius}" length="${pendulum_length}"/>
+          <mesh filename="package://pendulum_control/urdf/mesh/pendulum.stl" scale="0.001 0.001 0.001"/>
         </geometry>
       </collision>
       <!-- Inertia -->
-      <xacro:cyl_inertia mass="${pendulum_mass}" length="${pendulum_length}" radius="${pendulum_radius}"/>
+      <inertial>
+        <mass value="0.1"/>
+        <origin xyz="0 0 0" rpy="0 0 0"/>
+        <inertia ixx="0.001" ixy="0.0" ixz="0.0"
+                  iyy="0.001" iyz="0.0"
+                  izz="0.001"/>
+      </inertial>
     </link>
   </xacro:macro>

File: ros2_ws/src/pendulum_control/urdf/links/rotor_link.xacro (robot description, xacro)
@@ -1,8 +1,29 @@
 <?xml version="1.0"?>
 <robot xmlns:xacro="http://www.ros.org/wiki/xacro" name="link_macros">
-  <xacro:macro name="rotor_link" params="rotor_radius rotor_length rotor_mass">
+  <xacro:macro name="rotor_link" params="">
     <link name="rotor_link">
+      <!-- Visual -->
+      <visual>
+        <origin xyz="0 0 ${-rotor_height-pendulum_height}" rpy="0 0 0"/>
+        <geometry>
+          <mesh filename="package://pendulum_control/urdf/mesh/rotor.stl" scale="0.001 0.001 0.001"/>
+        </geometry>
+        <material name="red">
+          <color rgba="1 0 0 0.8"/>
+        </material>
+      </visual>
+      <!-- Collision -->
+      <Collision>
+        <origin xyz="0 0 0" rpy="0 0 0"/>
+        <mesh filename="pakcage://pendulum_control/urdf/mesh/rotor.stl" scale="0.001 0.001 0.001"/>
+      </Collision>
       <!-- Inertia -->
-      <xacro:cyl_inertia mass="${rotor_mass}" radius="${rotor_radius}" length="${rotor_length}"/>
+      <inertial>
+        <mass value="0.1"/>
+        <origin xyz="0 0 0" rpy="0 0 0"/>
+        <inertia ixx="0.001" ixy="0.0" ixz="0.0"
+                  iyy="0.001" iyz="0.0"
+                  izz="0.001"/>
+      </inertial>
     </link>
   </xacro:macro>

File: ros2_ws/src/pendulum_control/urdf/macros/inertia_macros.xacro (robot description, xacro)
@@ -14,8 +14,8 @@
     </inertial>
   </xacro:macro>
-  <xacro:macro name="base_inertia" params="mass">
+  <xacro:macro name="base_inertia" params="mass depth width height">
   <inertial>
     <mass value="${mass}"/>
-    <origin xyz="0 0 ${mass/2}" rpy="0 0 0"/>
+      <origin xyz="${depth/2} ${width/2} ${height/2}" rpy="0 0 0"/>
     <inertia ixx="${mass/6}" ixy="0" ixz="0" iyy="${mass/6}" iyz="0" izz="${mass/6}"/>
   </inertial>

File: ros2_ws/src/pendulum_control/urdf/qube_constants.xacro (robot description, xacro)
@@ -6,5 +6,5 @@
   <xacro:property name="base_mass" value="0.5"/>
   <xacro:property name="rotor_radius" value="0.00325"/>
-  <xacro:property name="rotor_length" value="0.085"/>
+  <xacro:property name="rotor_height" value="0.0104"/>
   <xacro:property name="rotor_mass" value="0.095"/>
   <xacro:property name="rotor_friction" value="0"/>
@@ -12,4 +12,5 @@
   <xacro:property name="pendulum_radius" value="0.0048"/>
   <xacro:property name="pendulum_length" value="0.129"/>
+  <xacro:property name="pendulum_height" value="0.01042"/>
   <xacro:property name="p_end_to_link" value="0.005"/>
   <xacro:property name="pendulum_mass" value="0.024"/>

File: ros2_ws/src/pendulum_control/urdf/qube_servo.urdf.xacro (robot description, xacro)
@@ -16,17 +16,7 @@
   <!-- links -->
   <xacro:world/>
-  <xacro:base_link
-      base_width="${base_width}"
-      base_depth="${base_depth}"
-      base_height="${base_height}"
-      base_mass="${base_mass}"/>
-  <xacro:rotor_link
-      rotor_radius="${rotor_radius}"
-      rotor_length="${rotor_length}"
-      rotor_mass="${rotor_mass}"/>
-  <xacro:pendulum_link
-      pendulum_radius="${pendulum_radius}"
-      pendulum_length="${pendulum_length}"
-      pendulum_mass="${pendulum_mass}"/>
+  <xacro:base_link/>
+  <xacro:rotor_link/>
+  <xacro:pendulum_link/>
   <!-- joints -->
   <xacro:base_joint/>

Commit message: gazebo +-145 fix. +- signs fliped. New sim paramaters added

File: ros2_ws/src/pendulum_control/urdf/joints/rotor_joint.xacro (robot description, xacro)
@@ -7,5 +7,5 @@
       <origin xyz="0 0 ${base_height+rotor_height+pendulum_height}" rpy="0 0 0"/>
       <axis xyz="0 0 1"/>
-      <limit effort="2" velocity="20" lower="-1.5708" upper="1.5708"/>
+      <limit effort="2" velocity="20" lower="-2.35619" upper="2.35619"/>
       <dynamics damping="${rotor_damping}" friction="${rotor_friction}"/>
     </joint>

Commit message: swing up looking good in simulation

File: ros2_ws/src/pendulum_control/urdf/joints/rotor_joint.xacro (robot description, xacro)
@@ -7,5 +7,5 @@
       <origin xyz="0 0 ${base_height+rotor_height+pendulum_height}" rpy="0 0 0"/>
       <axis xyz="0 0 1"/>
-      <limit effort="100" velocity="20" lower="-2.35619" upper="2.35619"/>
+      <limit effort="100" velocity="200" lower="-2.35619" upper="2.35619"/>
       <dynamics damping="${rotor_damping}" friction="${rotor_friction}"/>
     </joint>
