Commit message: Merge

File: ros2_ws/src/pendulum_control/urdf/joints/pendulum_joint.xacro (robot description, xacro)
@@ -1,10 +1,12 @@
 <?xml version="1.0"?>
-<robot xmlns:xacro="http://www.ros.org/wiki/xacro">
-<joint name="pendulum_joint" type="revolute">
-  <parent link="rotor_link"/>
-  <child link="pendulum_link"/>
-  <origin xyz="0 0 0" rpy="0 1.5708 0"/>
-  <axis xyz="0 1 0"/>
-  <limit effort="2" velocity="20" lower="-3.14" upper="3.14"/>
-</joint>
+<robot xmlns:xacro="http://www.ros.org/wiki/xacro" name="joint_macros">
+  <xacro:macro name="pendulum_joint" params="">
+    <joint name="pendulum_joint" type="revolute">
+      <parent link="rotor_link"/>
+      <child link="pendulum_link"/>
+      <origin xyz="0 0 ${rotor_radius}" rpy="0 1.5708 0"/>
+      <axis xyz="0 1 0"/>
+      <limit effort="2" velocity="20" lower="-3.14" upper="3.14"/>
+    </joint>
+  </xacro:macro>
 </robot>

File: ros2_ws/src/pendulum_control/urdf/joints/rotor_joint.xacro (robot description, xacro)
@@ -1,10 +1,12 @@
 <?xml version="1.0"?>
-<robot xmlns:xacro="http://www.ros.org/wiki/xacro">
-<joint name="rotor_joint" type="revolute">
-  <parent link="base_link"/>
-  <child link="rotor_link"/>
-  <origin xyz="0 0 0.058" rpy="0 0 0"/>
-  <axis xyz="0 0 1"/>
-  <limit effort="2" velocity="20" lower="-6.28" upper="6.28"/>
-</joint>
+<robot xmlns:xacro="http://www.ros.org/wiki/xacro" name="joint_macros">
+  <xacro:macro name="rotor_joint" params="">
+    <joint name="rotor_joint" type="revolute">
+      <parent link="base_link"/>
+      <child link="rotor_link"/>
+      <origin xyz="0 0 ${base_height}" rpy="0 0 0"/>
+      <axis xyz="0 0 1"/>
+      <limit effort="2" velocity="20" lower="-6.28" upper="6.28"/>
+    </joint>
+  </xacro:macro>
 </robot>

File: ros2_ws/src/pendulum_control/urdf/links/base_link.xacro (robot description, xacro)
@@ -1,16 +1,23 @@
 <?xml version="1.0"?>
-<robot xmlns:xacro="htpp://www.ros.org/wiki/xacro">
-<link name="base_link">
-  <visual>
-    <geometry>
-      <box size="${base_size} ${base_size} ${base_height}"/>
-    </geometry>
-  </visual>
-  <collision>
-    <geometry>
-      <box size="${base_size} ${base_size} ${base_height}"/>
-    </geometry>
-  </collision>
-  <xacro:simple_inertia mass="${base_mass}"/>
-</link>
+<robot xmlns:xacro="http://www.ros.org/wiki/xacro" name="link_macros">
+  <xacro:macro name="base_link" params="base_size base_height base_mass">
+    <link name="base_link">
+      <!-- Visual -->
+      <visual>
+        <origin xyz="0 0 ${base_height/2}" rpy="0 0 0"/>
+        <geometry>
+          <box size="${base_size} ${base_size} ${base_height}"/>
+        </geometry>
+      </visual>
+      <!-- Collision -->
+      <collision>
+        <origin xyz="0 0 ${base_height/2}" rpy="0 0 0"/>
+        <geometry>
+          <box size="${base_size} ${base_size} ${base_height}"/>
+        </geometry>
+      </collision>
+      <!-- Inertia -->
+      <xacro:base_inertia mass="${base_mass}"/>
+    </link>
+  </xacro:macro>
 </robot>

File: ros2_ws/src/pendulum_control/urdf/links/pendulum_link.xacro (robot description, xacro)
@@ -1,18 +1,23 @@
 <?xml version="1.0"?>
-<robot xmlns:xacro="http://www.ros.org/wiki/xacro">
-<link name="pendulum_link">
-  <visual>
-    <origin xyz="0 0 ${pendulum_length/2}"/>
-    <geometry>
-      <cylinder radius="${pendulum_radius}" length="${pendulum_length}"/>
-    </geometry>
-  </visual>
-  <collision>
-    <origin xyz="0 0 ${pendulum_length/2}"/>
-    <geometry>
-      <cylinder radius="${pendulum_radius}" length="${pendulum_length}"/>
-    </geometry>
-  </collision>
-  <xacro:simple_inertia mass="${pendulum_mass}"/>
-</link>
+<robot xmlns:xacro="http://www.ros.org/wiki/xacro" name="link_macros">
+  <xacro:macro name="pendulum_link" params="pendulum_radius pendulum_length pendulum_mass">
+    <link name="pendulum_link">
+      <!-- Visual -->
+      <visual>
+        <origin xyz="0 0 ${pendulum_length/2}" rpy="0 0 0"/>
+        <geometry>
+          <cylinder radius="${pendulum_radius}" length="${pendulum_length}"/>
+        </geometry>
+      </visual>
+      <!-- Collision -->
+      <collision>
+        <origin xyz="0 0 ${pendulum_length/2}" rpy="0 0 0"/>
+        <geometry>
+          <cylinder radius="${pendulum_radius}" length="${pendulum_length}"/>
+        </geometry>
+      </collision>
+      <!-- Inertia -->
+      <xacro:cyl_inertia mass="${pendulum_mass}" length="${pendulum_length}" radius="${pendulum_radius}"/>
+    </link>
+  </xacro:macro>
 </robot>

File: ros2_ws/src/pendulum_control/urdf/links/rotor_link.xacro (robot description, xacro)
@@ -1,16 +1,23 @@
 <?xml version="1.0"?>
-<robot xmlns:xacro="htpp://www.ros.org/wiki/xacro">
-<link name="rotor_link">
-  <visual>
-    <geometry>
-      <cylinder radius="${rotor_radius}" length="${rotor_length}"/>
-    </geometry>
-  </visual>
-  <collision>
-    <geometry>
-      <cylinder radius="${rotor_radius}" length="${rotor_length}"/>
-    </geometry>
-  </collision>
-  <xacro:simple_inertia mass="${rotor_mass}"/>
-</link>
+<robot xmlns:xacro="http://www.ros.org/wiki/xacro" name="link_macros">
+  <xacro:macro name="rotor_link" params="rotor_radius rotor_length rotor_mass">
+    <link name="rotor_link">
+      <!-- Visual -->
+      <visual>
+        <origin xyz="0 0 0" rpy="0 0 0"/>
+        <geometry>
+          <cylinder radius="${rotor_radius}" length="${rotor_length}"/>
+        </geometry>
+      </visual>
+      <!-- Collision -->
+      <collision>
+        <origin xyz="0 0 0" rpy="0 0 0"/>
+        <geometry>
+          <cylinder radius="${rotor_radius}" length="${rotor_length}"/>
+        </geometry>
+      </collision>
+      <!-- Inertia -->
+      <xacro:cyl_inertia mass="${rotor_mass}" radius="${rotor_radius}" length="${rotor_length}"/>
+    </link>
+  </xacro:macro>
 </robot>

File: ros2_ws/src/pendulum_control/urdf/macros/inertia_macros.xacro (robot description, xacro)
@@ -1,16 +1,23 @@
 <?xml version="1.0"?>
-<robot xmlns:xacro="http://www.ros.org/wiki/xacro">
-<xacro:macro name="simple_inertia" params="mass">
-<inertial>
-  <mass value="${mass}"/>
-  <origin xyz="0 0 0"/>
-  <inertia
-    ixx="0.001"
-    iyy="0.001"
-    izz="0.001"
-    ixy="0"
-    ixz="0"
-    iyz="0"/>
-</inertial>
-</xacro:macro>
+<robot xmlns:xacro="http://www.ros.org/wiki/xacro" name="inertia_macros">
+ <xacro:macro name="cyl_inertia" params="mass radius length">
+    <inertial>
+      <mass value="${mass}"/>
+      <!-- COM at geometric center -->
+      <origin xyz="0 0 0" rpy="0 0 0"/>
+      <inertia
+        ixx="${(1/12.0)*mass*length*length + 0.25*mass*radius*radius}"
+        ixy="0" ixz="0"
+        iyy="${(1/12.0)*mass*length*length + 0.25*mass*radius*radius}"
+        iyz="0"
+        izz="${0.5*mass*radius*radius}"/>
+    </inertial>
+  </xacro:macro>
+  <xacro:macro name="base_inertia" params="mass">
+  <inertial>
+    <mass value="${mass}"/>
+    <origin xyz="0 0 ${mass/2}" rpy="0 0 0"/>
+    <inertia ixx="${mass/6}" ixy="0" ixz="0" iyy="${mass/6}" iyz="0" izz="${mass/6}"/>
+  </inertial>
+  </xacro:macro>
 </robot>

File: ros2_ws/src/pendulum_control/urdf/qube_constants.xacro (robot description, xacro)
@@ -1,12 +1,12 @@
 <?xml version="1.0"?>
-<robot xmlns:xacro="http://www.ros.org/wiki/xacro">
-<xacro:property name="base_size" value="0.102"/>
-<xacro:property name="base_height" value="0.117"/>
-<xacro:property name="rotor_mass_radius" value="0.01"/>
-<xacro:property name="rotor_length" value="0.02"/>
-<xacro:property name="pendulum_radius" value="0.005"/>
-<xacro:property name="pendulum_length" value="0.095"/>
-<xacro:property name="base_mass" value="0.5"/>
-<xacro:property name="rotor_mass" value="0.05"/>
-<xacro:property name"pendulum_mass" value"0.02"/>
-</robot>
+<xacro:constants xmlns:xacro="http://www.ros.org/wiki/xacro">
+  <xacro:property name="base_size" value="0.102"/>
+  <xacro:property name="base_height" value="0.117"/>
+  <xacro:property name="base_mass" value="0.5"/>
+  <xacro:property name="rotor_radius" value="0.01"/>
+  <xacro:property name="rotor_length" value="0.02"/>
+  <xacro:property name="rotor_mass" value="0.05"/>
+  <xacro:property name="pendulum_radius" value="0.005"/>
+  <xacro:property name="pendulum_length" value="0.095"/>
+  <xacro:property name="pendulum_mass" value="0.02"/>
+</xacro:constants>

File: ros2_ws/src/pendulum_control/urdf/qube_servo.urdf.xacro (robot description, xacro)
@@ -1,14 +1,33 @@
 <?xml version="1.0"?>
 <robot name="qube_servo_3" xmlns:xacro="http://www.ros.org/wiki/xacro">
-<!-- constants -->
-<xacro:include filename="$(find pendulum_control)/urdf/qube_constants.xacro"/>
-<!-- macros -->
-<xacro:include filename="$(find pendulum_control)/urdf/macros/inertia_macros.xacro"/>
-<!-- links -->
-<xacro:include filename="$(find pendulum_control)/urdf/links/base_link.xacro"/>
-<xacro:include filename="$(find pendulum_control)/urdf/links/rotor_link.xacro"/>
-<xacro:include filename="$(find pendulum_control)/urdf/links/pendulum_link.xacro"/>
-<!-- joints -->
-<xacro:include filename="$(find pendulum_control)/urdf/joints/rotor_joint.xacro"/>
-<xacro:include filename="$/find pendulum_control)/urdf/joints/pendulum_joint.xacro"/>
+  <!-- constants -->
+  <xacro:include filename="$(find pendulum_control)/urdf/qube_constants.xacro"/>
+  <!-- inertias -->
+  <xacro:include filename="$(find pendulum_control)/urdf/macros/inertia_macros.xacro"/>
+  <!-- links -->
+  <xacro:include filename="$(find pendulum_control)/urdf/links/world.xacro"/>
+  <xacro:include filename="$(find pendulum_control)/urdf/links/base_link.xacro"/>
+  <xacro:include filename="$(find pendulum_control)/urdf/links/rotor_link.xacro"/>
+  <xacro:include filename="$(find pendulum_control)/urdf/links/pendulum_link.xacro"/>
+  <!-- joints -->
+  <xacro:include filename="$(find pendulum_control)/urdf/joints/base_joint.xacro"/>
+  <xacro:include filename="$(find pendulum_control)/urdf/joints/rotor_joint.xacro"/>
+  <xacro:include filename="$(find pendulum_control)/urdf/joints/pendulum_joint.xacro"/>
+  <!-- expand macros with parameters -->
+  <xacro:world/>
+  <xacro:base_link
+      base_size="${base_size}"
+      base_height="${base_height}"
+      base_mass="${base_mass}"/>
+  <xacro:rotor_link
+      rotor_radius="${rotor_radius}"
+      rotor_length="${rotor_length}"
+      rotor_mass="${rotor_mass}"/>
+  <xacro:pendulum_link
+      pendulum_radius="${pendulum_radius}"
+      pendulum_length="${pendulum_length}"
+      pendulum_mass="${pendulum_mass}"/>
+  <xacro:base_joint/>
+  <xacro:rotor_joint/>
+  <xacro:pendulum_joint/>
 </robot>

Commit message: rough URDF file

File: ros2_ws/src/pendulum_control/urdf/joints/pendulum_joint.xacro (robot description, xacro)
@@ -5,6 +5,6 @@
       <parent link="rotor_link"/>
       <child link="pendulum_link"/>
-      <origin xyz="0 0 ${rotor_radius}" rpy="0 1.5708 0"/>
-      <axis xyz="0 1 0"/>
+      <origin xyz="${rotor_length} 0 0" rpy="0 1.5708 0"/>
+      <axis xyz="0 0 1"/>
       <limit effort="2" velocity="20" lower="-3.14" upper="3.14"/>
     </joint>

File: ros2_ws/src/pendulum_control/urdf/joints/rotor_joint.xacro (robot description, xacro)
@@ -5,7 +5,7 @@
       <parent link="base_link"/>
       <child link="rotor_link"/>
-      <origin xyz="0 0 ${base_height}" rpy="0 0 0"/>
+      <origin xyz="0 0 ${base_height+rotor_radius}" rpy="0 0 0"/>
       <axis xyz="0 0 1"/>
-      <limit effort="2" velocity="20" lower="-6.28" upper="6.28"/>
+      <limit effort="2" velocity="20" lower="-1.5708" upper="1.5708"/>
     </joint>
   </xacro:macro>

File: ros2_ws/src/pendulum_control/urdf/links/base_link.xacro (robot description, xacro)
@@ -1,5 +1,5 @@
 <?xml version="1.0"?>
 <robot xmlns:xacro="http://www.ros.org/wiki/xacro" name="link_macros">
-  <xacro:macro name="base_link" params="base_size base_height base_mass">
+  <xacro:macro name="base_link" params="base_width base_depth base_height base_mass">
     <link name="base_link">
       <!-- Visual -->
@@ -7,5 +7,5 @@
         <origin xyz="0 0 ${base_height/2}" rpy="0 0 0"/>
         <geometry>
-          <box size="${base_size} ${base_size} ${base_height}"/>
+          <box size="${base_width} ${base_depth} ${base_height}"/>
         </geometry>
       </visual>
@@ -14,5 +14,5 @@
         <origin xyz="0 0 ${base_height/2}" rpy="0 0 0"/>
         <geometry>
-          <box size="${base_size} ${base_size} ${base_height}"/>
+          <box size="${base_width} ${base_depth} ${base_height}"/>
         </geometry>
       </collision>

File: ros2_ws/src/pendulum_control/urdf/links/pendulum_link.xacro (robot description, xacro)
@@ -5,12 +5,15 @@
       <!-- Visual -->
       <visual>
-        <origin xyz="0 0 ${pendulum_length/2}" rpy="0 0 0"/>
+        <origin xyz="${pendulum_length/2} 0 0" rpy="0 1.5708 0"/>
         <geometry>
           <cylinder radius="${pendulum_radius}" length="${pendulum_length}"/>
         </geometry>
+        <material name="orange">
+          <color rgba="1 0.65 0 0.8"/>
+        </material>
       </visual>
       <!-- Collision -->
       <collision>
-        <origin xyz="0 0 ${pendulum_length/2}" rpy="0 0 0"/>
+        <origin xyz="0 0 0" rpy="0 0 0"/>
         <geometry>
           <cylinder radius="${pendulum_radius}" length="${pendulum_length}"/>

File: ros2_ws/src/pendulum_control/urdf/links/rotor_link.xacro (robot description, xacro)
@@ -5,12 +5,15 @@
       <!-- Visual -->
       <visual>
-        <origin xyz="0 0 0" rpy="0 0 0"/>
+        <origin xyz="${rotor_length/2} 0 0" rpy="0 1.5708 0"/>
         <geometry>
           <cylinder radius="${rotor_radius}" length="${rotor_length}"/>
         </geometry>
+        <material name="green">
+          <color rgba="0 1 0 0.8"/>
+        </material>
       </visual>
       <!-- Collision -->
       <collision>
-        <origin xyz="0 0 0" rpy="0 0 0"/>
+        <origin xyz="0 0 0" rpy="0 1.5708 0"/>
         <geometry>
           <cylinder radius="${rotor_radius}" length="${rotor_length}"/>

File: ros2_ws/src/pendulum_control/urdf/qube_constants.xacro (robot description, xacro)
@@ -1,12 +1,13 @@
 <?xml version="1.0"?>
 <xacro:constants xmlns:xacro="http://www.ros.org/wiki/xacro">
-  <xacro:property name="base_size" value="0.102"/>
-  <xacro:property name="base_height" value="0.117"/>
+  <xacro:property name="base_width" value="0.102"/>
+  <xacro:property name="base_height" value="0.102"/>
+  <xacro:property name="base_depth" value="0.117"/>
   <xacro:property name="base_mass" value="0.5"/>
   <xacro:property name="rotor_radius" value="0.01"/>
-  <xacro:property name="rotor_length" value="0.02"/>
-  <xacro:property name="rotor_mass" value="0.05"/>
+  <xacro:property name="rotor_length" value="0.085"/>
+  <xacro:property name="rotor_mass" value="0.095"/>
   <xacro:property name="pendulum_radius" value="0.005"/>
-  <xacro:property name="pendulum_length" value="0.095"/>
-  <xacro:property name="pendulum_mass" value="0.02"/>
+  <xacro:property name="pendulum_length" value="0.129"/>
+  <xacro:property name="pendulum_mass" value="0.024"/>
 </xacro:constants>

File: ros2_ws/src/pendulum_control/urdf/qube_servo.urdf.xacro (robot description, xacro)
@@ -17,5 +17,6 @@
   <xacro:world/>
   <xacro:base_link
-      base_size="${base_size}"
+      base_width="${base_width}"
+      base_depth="${base_depth}"
       base_height="${base_height}"
       base_mass="${base_mass}"/>

Commit message: Setup gazebo and controller interface

File: ros2_ws/src/pendulum_control/urdf/joints/pendulum_joint.xacro (robot description, xacro)
@@ -2,10 +2,11 @@
 <robot xmlns:xacro="http://www.ros.org/wiki/xacro" name="joint_macros">
   <xacro:macro name="pendulum_joint" params="">
-    <joint name="pendulum_joint" type="revolute">
+    <joint name="pendulum_joint" type="continuous">
       <parent link="rotor_link"/>
       <child link="pendulum_link"/>
       <origin xyz="${rotor_length} 0 0" rpy="0 1.5708 0"/>
       <axis xyz="0 0 1"/>
-      <limit effort="2" velocity="20" lower="-3.14" upper="3.14"/>
+      <limit effort="2" velocity="20"/>
+      <dynamics damping="0" friction="0"/>
     </joint>
   </xacro:macro>

File: ros2_ws/src/pendulum_control/urdf/joints/rotor_joint.xacro (robot description, xacro)
@@ -8,4 +8,5 @@
       <axis xyz="0 0 1"/>
       <limit effort="2" velocity="20" lower="-1.5708" upper="1.5708"/>
+      <dynamics damping="0.05" friction="0.01"/>
     </joint>
   </xacro:macro>

File: ros2_ws/src/pendulum_control/urdf/qube_servo.urdf.xacro (robot description, xacro)
@@ -14,5 +14,5 @@
   <xacro:include filename="$(find pendulum_control)/urdf/joints/rotor_joint.xacro"/>
   <xacro:include filename="$(find pendulum_control)/urdf/joints/pendulum_joint.xacro"/>
-  <!-- expand macros with parameters -->
+  <!-- links -->
   <xacro:world/>
   <xacro:base_link
@@ -29,6 +29,45 @@
       pendulum_length="${pendulum_length}"
       pendulum_mass="${pendulum_mass}"/>
+  <!-- joints -->
   <xacro:base_joint/>
   <xacro:rotor_joint/>
   <xacro:pendulum_joint/>
+  <!-- ros2 controll hardware interface -->
+  <ros2_control name="GazeboSystem" type="System">
+    <hardware>
+      <plugin>gz_ros2_control/GazeboSimSystem</plugin>
+    </hardware>
+    <joint name="rotor_joint">
+      <command_interface name="effort"/>
+      <state_interface name="position"/>
+      <state_interface name="velocity"/>
+    </joint>
+    <joint name="pendulum_joint">
+      <state_interface name="position"/>
+      <state_interface name="velocity"/>
+    </joint>
+  </ros2_control>
+  <!-- gazebo plugins -->
+  <gazebo>
+    <plugin filename="libgz_ros2_control-system.so" name="gz_ros2_control::GazeboSimROS2ControlPlugin">
+      <parameters>$(find pendulum_control)/config/controllers.yaml</parameters>
+    </plugin>
+  </gazebo>
+  <!-- gazebo materials -->
+  <gazebo reference="base_link">
+    <material>Gazebo/Red</material>
+  </gazebo>
+  <gazebo reference="rotor_link">
+    <material>Gazebo/Green</material>
+  </gazebo>
+  <gazebo reference="pendulum_link">
+    <material>Gazebo/Orange</material>
+  </gazebo>
+  <!-- joint dynamics -->
+  <gazebo reference="rotor_joint">
+    <implicitSpringDamper>true</implicitSpringDamper>
+  </gazebo>
+  <gazebo reference="pendulum_joint">
+    <implicitSpringDamper>true</implicitSpringDamper>
+  </gazebo>
 </robot>

Commit message: Added constants for joint friction and dampning

File: ros2_ws/src/pendulum_control/urdf/joints/pendulum_joint.xacro (robot description, xacro)
@@ -8,5 +8,5 @@
       <axis xyz="0 0 1"/>
       <limit effort="2" velocity="20"/>
-      <dynamics damping="0" friction="0"/>
+      <dynamics damping="${pendulum_damping}" friction="${pendulum_friction}"/>
     </joint>
   </xacro:macro>

File: ros2_ws/src/pendulum_control/urdf/joints/rotor_joint.xacro (robot description, xacro)
@@ -8,5 +8,5 @@
       <axis xyz="0 0 1"/>
       <limit effort="2" velocity="20" lower="-1.5708" upper="1.5708"/>
-      <dynamics damping="0.05" friction="0.01"/>
+      <dynamics damping="${rotor_damping}" friction="${rotor_friction}"/>
     </joint>
   </xacro:macro>

File: ros2_ws/src/pendulum_control/urdf/qube_constants.xacro (robot description, xacro)
@@ -8,6 +8,10 @@
   <xacro:property name="rotor_length" value="0.085"/>
   <xacro:property name="rotor_mass" value="0.095"/>
+  <xacro:property name="rotor_friction" value="0.01"/>
+  <xacro:property name="rotor_damping" value="0.05"/>
   <xacro:property name="pendulum_radius" value="0.005"/>
   <xacro:property name="pendulum_length" value="0.129"/>
   <xacro:property name="pendulum_mass" value="0.024"/>
+  <xacro:property name="pendulum_friction" value="0"/>
+  <xacro:property name="pendulum_damping" value="0"/>
 </xacro:constants>

Commit message: Correct joint specification

File: ros2_ws/src/pendulum_control/urdf/joints/pendulum_joint.xacro (robot description, xacro)
@@ -5,5 +5,5 @@
       <parent link="rotor_link"/>
       <child link="pendulum_link"/>
-      <origin xyz="${rotor_length} 0 0" rpy="0 1.5708 0"/>
+      <origin xyz="0 0 0" rpy="0 1.5708 0"/>
       <axis xyz="0 0 1"/>
       <limit effort="2" velocity="20"/>

File: ros2_ws/src/pendulum_control/urdf/links/base_link.xacro (robot description, xacro)
@@ -7,5 +7,5 @@
         <origin xyz="0 0 ${base_height/2}" rpy="0 0 0"/>
         <geometry>
-          <box size="${base_width} ${base_depth} ${base_height}"/>
+          <box size="${base_depth} ${base_width} ${base_height}"/>
         </geometry>
       </visual>

File: ros2_ws/src/pendulum_control/urdf/links/pendulum_link.xacro (robot description, xacro)
@@ -5,10 +5,19 @@
       <!-- Visual -->
       <visual>
-        <origin xyz="${pendulum_length/2} 0 0" rpy="0 1.5708 0"/>
+        <origin xyz="0 0 ${rotor_length/2}" rpy="0 0 0"/>
+        <geometry>
+          <cylinder radius="${rotor_radius}" length="${rotor_length}"/>
+        </geometry>
+        <material name="green">
+          <color rgba="0 1 0 0.8"/>
+        </material>
+      </visual>
+      <visual>
+        <origin xyz="${pendulum_length/2-p_end_to_link-rotor_radius} 0 ${rotor_length-pendulum_radius/2}" rpy="0 1.5708 0"/>
         <geometry>
           <cylinder radius="${pendulum_radius}" length="${pendulum_length}"/>
         </geometry>
         <material name="orange">
-          <color rgba="1 0.65 0 0.8"/>
+          <color rbga="1 0.65 0 0.8"/>
         </material>
       </visual>

File: ros2_ws/src/pendulum_control/urdf/links/rotor_link.xacro (robot description, xacro)
@@ -3,21 +3,4 @@
   <xacro:macro name="rotor_link" params="rotor_radius rotor_length rotor_mass">
     <link name="rotor_link">
-      <!-- Visual -->
-      <visual>
-        <origin xyz="${rotor_length/2} 0 0" rpy="0 1.5708 0"/>
-        <geometry>
-          <cylinder radius="${rotor_radius}" length="${rotor_length}"/>
-        </geometry>
-        <material name="green">
-          <color rgba="0 1 0 0.8"/>
-        </material>
-      </visual>
-      <!-- Collision -->
-      <collision>
-        <origin xyz="0 0 0" rpy="0 1.5708 0"/>
-        <geometry>
-          <cylinder radius="${rotor_radius}" length="${rotor_length}"/>
-        </geometry>
-      </collision>
       <!-- Inertia -->
       <xacro:cyl_inertia mass="${rotor_mass}" radius="${rotor_radius}" length="${rotor_length}"/>

File: ros2_ws/src/pendulum_control/urdf/qube_constants.xacro (robot description, xacro)
@@ -5,11 +5,12 @@
   <xacro:property name="base_depth" value="0.117"/>
   <xacro:property name="base_mass" value="0.5"/>
-  <xacro:property name="rotor_radius" value="0.01"/>
+  <xacro:property name="rotor_radius" value="0.0065"/>
   <xacro:property name="rotor_length" value="0.085"/>
   <xacro:property name="rotor_mass" value="0.095"/>
   <xacro:property name="rotor_friction" value="0"/>
   <xacro:property name="rotor_damping" value="0"/>
-  <xacro:property name="pendulum_radius" value="0.005"/>
+  <xacro:property name="pendulum_radius" value="0.0096"/>
   <xacro:property name="pendulum_length" value="0.129"/>
+  <xacro:property name="p_end_to_link" value="0.005"/>
   <xacro:property name="pendulum_mass" value="0.024"/>
   <xacro:property name="pendulum_friction" value="0"/>
