Commit message: Simulation closer to working

File: ros2_ws/src/pendulum_control/urdf/joints/pendulum_joint.xacro (robot description, xacro)
@@ -7,5 +7,5 @@
       <origin xyz="0 0 0" rpy="0 1.5708 0"/>
       <axis xyz="0 0 1"/>
-      <limit effort="2" velocity="20"/>
+      <limit effort="100" velocity="20"/>
       <dynamics damping="${pendulum_damping}" friction="${pendulum_friction}"/>
     </joint>

File: ros2_ws/src/pendulum_control/urdf/joints/rotor_joint.xacro (robot description, xacro)
@@ -7,5 +7,5 @@
       <origin xyz="0 0 ${base_height+rotor_height+pendulum_height}" rpy="0 0 0"/>
       <axis xyz="0 0 1"/>
-      <limit effort="2" velocity="20" lower="-2.35619" upper="2.35619"/>
+      <limit effort="100" velocity="20" lower="-2.35619" upper="2.35619"/>
       <dynamics damping="${rotor_damping}" friction="${rotor_friction}"/>
     </joint>

Commit message: Update pendulum and rotor link parameters for improved dynamics and inertia calculations

File: ros2_ws/src/pendulum_control/urdf/joints/pendulum_joint.xacro (robot description, xacro)
@@ -5,5 +5,5 @@
       <parent link="rotor_link"/>
       <child link="pendulum_link"/>
-      <origin xyz="0 0 0" rpy="0 1.5708 0"/>
+    <origin xyz="0.045427 0 0" rpy="0 0 0"/>
       <axis xyz="0 0 1"/>
       <limit effort="2" velocity="20"/>

File: ros2_ws/src/pendulum_control/urdf/links/pendulum_link.xacro (robot description, xacro)
@@ -22,13 +22,13 @@
       <!-- Inertia -->
      <inertial>
-        <origin xyz="0.0130 0 0.0511" rpy="0 0 0"/>
+      <origin xyz="0.045427 0 -0.0113445" rpy="0 0 0"/>
         <mass value="0.119"/>
         <inertia
-          ixx="9.20e-5"
-          ixy="0"
-          ixz="-5.25e-5"
-          iyy="2.05e-4"
-          iyz="0"
-          izz="1.14e-4"/>
+        ixx="9.8995e-5"
+        ixy="0"
+        ixz="0"
+        iyy="9.8995e-5"
+        iyz="0"
+        izz="9.8995e-5"/>
      </inertial>
     </link>

File: ros2_ws/src/pendulum_control/urdf/links/rotor_link.xacro (robot description, xacro)
@@ -23,10 +23,10 @@
       <mass value="0.0106"/>
        <inertia
-          ixx="1.4e-6"
-          ixy="0"
-          ixz="0"
-          iyy="1.4e-6"
-          iyz="0"
-          izz="1.4e-6"/>
+        ixx="1e-6"
+        ixy="0"
+        ixz="0"
+        iyy="1e-6"
+        iyz="0"
+        izz="0.0003716"/>
       </inertial>
     </link>

Commit message: Refine pendulum and rotor joint parameters for improved simulation accuracy

File: ros2_ws/src/pendulum_control/urdf/joints/pendulum_joint.xacro (robot description, xacro)
@@ -5,7 +5,7 @@
       <parent link="rotor_link"/>
       <child link="pendulum_link"/>
-      <origin xyz="0 0 0" rpy="0 1.5708 0"/>
+    <origin xyz="0.045427 0 0" rpy="0 0 0"/>
       <axis xyz="0 0 1"/>
-      <limit effort="100" velocity="20"/>
+      <limit effort="2" velocity="20"/>
       <dynamics damping="${pendulum_damping}" friction="${pendulum_friction}"/>
     </joint>

File: ros2_ws/src/pendulum_control/urdf/joints/rotor_joint.xacro (robot description, xacro)
@@ -7,5 +7,5 @@
       <origin xyz="0 0 ${base_height+rotor_height+pendulum_height}" rpy="0 0 0"/>
       <axis xyz="0 0 1"/>
-      <limit effort="100" velocity="200" lower="-2.35619" upper="2.35619"/>
+      <limit effort="2" velocity="20" lower="-2.35619" upper="2.35619"/>
       <dynamics damping="${rotor_damping}" friction="${rotor_friction}"/>
     </joint>

File: ros2_ws/src/pendulum_control/urdf/links/rotor_link.xacro (robot description, xacro)
@@ -23,10 +23,10 @@
       <mass value="0.0106"/>
        <inertia
-          ixx="0.0003716"
-          ixy="0"
-          ixz="0"
-          iyy="0.0003716"
-          iyz="0"
-          izz="0.0003716"/>
+        ixx="1e-6"
+        ixy="0"
+        ixz="0"
+        iyy="1e-6"
+        iyz="0"
+        izz="0.0003716"/>
       </inertial>
     </link>

Commit message: Revert "Refine pendulum and rotor joint parameters for improved simulation accuracy"
This reverts commit 8b15b204158f8bdb03679f6dca5362cbbe5687ec.

File: ros2_ws/src/pendulum_control/urdf/joints/pendulum_joint.xacro (robot description, xacro)
@@ -5,7 +5,7 @@
       <parent link="rotor_link"/>
       <child link="pendulum_link"/>
-    <origin xyz="0.045427 0 0" rpy="0 0 0"/>
+      <origin xyz="0 0 0" rpy="0 1.5708 0"/>
       <axis xyz="0 0 1"/>
-      <limit effort="2" velocity="20"/>
+      <limit effort="100" velocity="20"/>
       <dynamics damping="${pendulum_damping}" friction="${pendulum_friction}"/>
     </joint>

File: ros2_ws/src/pendulum_control/urdf/joints/rotor_joint.xacro (robot description, xacro)
@@ -7,5 +7,5 @@
       <origin xyz="0 0 ${base_height+rotor_height+pendulum_height}" rpy="0 0 0"/>
       <axis xyz="0 0 1"/>
-      <limit effort="2" velocity="20" lower="-2.35619" upper="2.35619"/>
+      <limit effort="100" velocity="200" lower="-2.35619" upper="2.35619"/>
       <dynamics damping="${rotor_damping}" friction="${rotor_friction}"/>
     </joint>

File: ros2_ws/src/pendulum_control/urdf/links/pendulum_link.xacro (robot description, xacro)
@@ -22,13 +22,13 @@
       <!-- Inertia -->
      <inertial>
-      <origin xyz="0.045427 0 -0.0113445" rpy="0 0 0"/>
+        <origin xyz="0.0130 0 0.0511" rpy="0 0 0"/>
         <mass value="0.119"/>
         <inertia
-        ixx="9.8995e-5"
-        ixy="0"
-        ixz="0"
-        iyy="9.8995e-5"
-        iyz="0"
-        izz="9.8995e-5"/>
+          ixx="9.20e-5"
+          ixy="0"
+          ixz="-5.25e-5"
+          iyy="2.05e-4"
+          iyz="0"
+          izz="1.14e-4"/>
      </inertial>
     </link>

File: ros2_ws/src/pendulum_control/urdf/links/rotor_link.xacro (robot description, xacro)
@@ -23,10 +23,10 @@
       <mass value="0.0106"/>
        <inertia
-        ixx="1e-6"
-        ixy="0"
-        ixz="0"
-        iyy="1e-6"
-        iyz="0"
-        izz="0.0003716"/>
+          ixx="0.0003716"
+          ixy="0"
+          ixz="0"
+          iyy="0.0003716"
+          iyz="0"
+          izz="0.0003716"/>
       </inertial>
     </link>
