Commit message: fix inertia and color

File: ros2_ws/src/pendulum_control/urdf/links/rotor_link.xacro (robot description, xacro)
@@ -21,13 +21,13 @@
     <inertial>
       <origin xyz="0 0 0" rpy="0 0 0"/>
-      <mass value="${rotor_mass}"/>
-      <inertia
-        ixx="1.0e-6"
-        ixy="0"
-        ixz="0"
-        iyy="1.0e-6"
-        iyz="0"
-        izz="2.0e-6"/>
-    </inertial>
+      <mass value="0.0106"/>
+       <inertia
+          ixx="1.4e-6"
+          ixy="0"
+          ixz="0"
+          iyy="1.4e-6"
+          iyz="0"
+          izz="1.4e-6"/>
+      </inertial>
     </link>
   </xacro:macro>

File: ros2_ws/src/pendulum_control/urdf/qube_servo.urdf.xacro (robot description, xacro)
@@ -46,8 +46,8 @@
   <!-- gazebo materials -->
   <gazebo reference="base_link">
-    <material>Gazebo/Red</material>
+    <material>Gazebo/Green</material>
   </gazebo>
   <gazebo reference="rotor_link">
-    <material>Gazebo/Green</material>
+    <material>Gazebo/Red</material>
   </gazebo>
   <gazebo reference="pendulum_link">

Commit message: lukas values

File: ros2_ws/src/pendulum_control/urdf/links/rotor_link.xacro (robot description, xacro)
@@ -23,10 +23,10 @@
       <mass value="0.0106"/>
        <inertia
-          ixx="1.4e-6"
+          ixx="0.001486"
           ixy="0"
           ixz="0"
-          iyy="1.4e-6"
+          iyy="0.001486"
           iyz="0"
-          izz="1.4e-6"/>
+          izz="0.001486"/>
       </inertial>
     </link>

File: ros2_ws/src/pendulum_control/urdf/qube_constants.xacro (robot description, xacro)
@@ -8,6 +8,6 @@
   <xacro:property name="rotor_height" value="0.0104"/>
   <xacro:property name="rotor_mass" value="0.095"/>
-  <xacro:property name="rotor_friction" value="0"/>
-  <xacro:property name="rotor_damping" value="0.0001"/>
+  <xacro:property name="rotor_friction" value="0.0"/>
+  <xacro:property name="rotor_damping" value="0.001486"/>
   <xacro:property name="pendulum_radius" value="0.0048"/>
   <xacro:property name="pendulum_length" value="0.129"/>

Commit message: lukas nye tal v2

File: ros2_ws/src/pendulum_control/urdf/links/rotor_link.xacro (robot description, xacro)
@@ -23,10 +23,10 @@
       <mass value="0.0106"/>
        <inertia
-          ixx="0.001486"
+          ixx="0.0003716"
           ixy="0"
           ixz="0"
-          iyy="0.001486"
+          iyy="0.0003716"
           iyz="0"
-          izz="0.001486"/>
+          izz="0.0003716"/>
       </inertial>
     </link>

File: ros2_ws/src/pendulum_control/urdf/qube_constants.xacro (robot description, xacro)
@@ -9,5 +9,5 @@
   <xacro:property name="rotor_mass" value="0.095"/>
   <xacro:property name="rotor_friction" value="0.0"/>
-  <xacro:property name="rotor_damping" value="0.001486"/>
+  <xacro:property name="rotor_damping" value="3.611e-5"/>
   <xacro:property name="pendulum_radius" value="0.0048"/>
   <xacro:property name="pendulum_length" value="0.129"/>
