Commit message: inertia attempt

File: ros2_ws/src/pendulum_control/urdf/links/pendulum_link.xacro (robot description, xacro)
@@ -22,4 +22,5 @@
       <!-- Inertia -->
       <inertial>
+<<<<<<< Updated upstream
         <mass value="0.1"/>
         <origin xyz="0 0 0" rpy="0 0 0"/>
@@ -28,4 +29,16 @@
                   izz="0.001"/>
       </inertial>
+=======
+        <origin xyz="0.0130 0 0.0511" rpy="0 0 0"/>
+        <mass value="0.119"/>
+        <inertia
+          ixx="9.18e-5"
+          ixy="0"
+          ixz="-5.25e-5"
+          iyy="2.05e-4"
+          iyz="0"
+          izz="1.13e-4"/>
+      </inertial>
+>>>>>>> Stashed changes
     </link>
   </xacro:macro>

File: ros2_ws/src/pendulum_control/urdf/links/rotor_link.xacro (robot description, xacro)
@@ -19,4 +19,5 @@
       </Collision>
       <!-- Inertia -->
+<<<<<<< Updated upstream
       <inertial>
         <mass value="0.1"/>
@@ -26,5 +27,18 @@
                   izz="0.001"/>
       </inertial>
+=======
+    <inertial>
+      <origin xyz="0 0 0" rpy="0 0 0"/>
+      <mass value="${motor_mass}"/>
+      <inertia
+        ixx="1.0e-6"
+        ixy="0"
+        ixz="0"
+        iyy="1.0e-6"
+        iyz="0"
+        izz="2.0e-6"/>
+    </inertial>
+>>>>>>> Stashed changes
     </link>
   </xacro:macro>
-</robot>
+  </robot>

Commit message: inertia first attept

File: ros2_ws/src/pendulum_control/urdf/links/pendulum_link.xacro (robot description, xacro)
@@ -21,24 +21,15 @@
       </collision>
       <!-- Inertia -->
-      <inertial>
-<<<<<<< Updated upstream
-        <mass value="0.1"/>
-        <origin xyz="0 0 0" rpy="0 0 0"/>
-        <inertia ixx="0.001" ixy="0.0" ixz="0.0"
-                  iyy="0.001" iyz="0.0"
-                  izz="0.001"/>
-      </inertial>
-=======
+     <inertial>
         <origin xyz="0.0130 0 0.0511" rpy="0 0 0"/>
         <mass value="0.119"/>
         <inertia
-          ixx="9.18e-5"
+          ixx="9.20e-5"
           ixy="0"
           ixz="-5.25e-5"
           iyy="2.05e-4"
           iyz="0"
-          izz="1.13e-4"/>
-      </inertial>
->>>>>>> Stashed changes
+          izz="1.14e-4"/>
+     </inertial>
     </link>
   </xacro:macro>

File: ros2_ws/src/pendulum_control/urdf/links/rotor_link.xacro (robot description, xacro)
@@ -19,16 +19,7 @@
       </Collision>
       <!-- Inertia -->
-<<<<<<< Updated upstream
-      <inertial>
-        <mass value="0.1"/>
-        <origin xyz="0 0 0" rpy="0 0 0"/>
-        <inertia ixx="0.001" ixy="0.0" ixz="0.0"
-                  iyy="0.001" iyz="0.0"
-                  izz="0.001"/>
-      </inertial>
-=======
     <inertial>
       <origin xyz="0 0 0" rpy="0 0 0"/>
-      <mass value="${motor_mass}"/>
+      <mass value="${rotor_mass}"/>
       <inertia
         ixx="1.0e-6"
@@ -39,5 +30,4 @@
         izz="2.0e-6"/>
     </inertial>
->>>>>>> Stashed changes
     </link>
   </xacro:macro>

File: ros2_ws/src/pendulum_control/urdf/qube_constants.xacro (robot description, xacro)
@@ -9,5 +9,5 @@
   <xacro:property name="rotor_mass" value="0.095"/>
   <xacro:property name="rotor_friction" value="0"/>
-  <xacro:property name="rotor_damping" value="0"/>
+  <xacro:property name="rotor_damping" value="0.0001"/>
   <xacro:property name="pendulum_radius" value="0.0048"/>
   <xacro:property name="pendulum_length" value="0.129"/>

Commit message: Gazebo a little closer

File: ros2_ws/src/pendulum_control/urdf/links/pendulum_link.xacro (robot description, xacro)
@@ -23,5 +23,5 @@
      <inertial>
         <origin xyz="0.0130 0 0.0511" rpy="0 0 0"/>
-        <mass value="0.119"/>
+        <mass value="${pendulum_mass}"/>
         <inertia
           ixx="9.20e-5"

File: ros2_ws/src/pendulum_control/urdf/links/rotor_link.xacro (robot description, xacro)
@@ -14,12 +14,12 @@
       </visual>
       <!-- Collision -->
-      <Collision>
+      <collision>
         <origin xyz="0 0 0" rpy="0 0 0"/>
-        <mesh filename="pakcage://pendulum_control/urdf/mesh/rotor.stl" scale="0.001 0.001 0.001"/>
-      </Collision>
+        <mesh filename="package://pendulum_control/urdf/mesh/rotor.stl" scale="0.001 0.001 0.001"/>
+      </collision>
       <!-- Inertia -->
     <inertial>
       <origin xyz="0 0 0" rpy="0 0 0"/>
-      <mass value="0.0106"/>
+        <mass value="${rotor_mass}"/>
        <inertia
           ixx="0.0003716"

Commit message: Restore urdf file

File: ros2_ws/src/pendulum_control/urdf/links/pendulum_link.xacro (robot description, xacro)
@@ -22,13 +22,13 @@
       <!-- Inertia -->
      <inertial>
-      <origin xyz="0.045427 0 -0.0113445" rpy="0 0 0"/>
-        <mass value="0.119"/>
+        <origin xyz="0.0130 0 0.0511" rpy="0 0 0"/>
+        <mass value="${pendulum_mass}"/>
         <inertia
-        ixx="9.8995e-5"
-        ixy="0"
-        ixz="0"
-        iyy="9.8995e-5"
-        iyz="0"
-        izz="9.8995e-5"/>
+          ixx="9.20e-5"
+          ixy="0"
+          ixz="-5.25e-5"
+          iyy="2.05e-4"
+          iyz="0"
+          izz="1.14e-4"/>
      </inertial>
     </link>

File: ros2_ws/src/pendulum_control/urdf/links/rotor_link.xacro (robot description, xacro)
@@ -14,19 +14,19 @@
       </visual>
       <!-- Collision -->
-      <Collision>
+      <collision>
         <origin xyz="0 0 0" rpy="0 0 0"/>
-        <mesh filename="pakcage://pendulum_control/urdf/mesh/rotor.stl" scale="0.001 0.001 0.001"/>
-      </Collision>
+        <mesh filename="package://pendulum_control/urdf/mesh/rotor.stl" scale="0.001 0.001 0.001"/>
+      </collision>
       <!-- Inertia -->
     <inertial>
       <origin xyz="0 0 0" rpy="0 0 0"/>
-      <mass value="0.0106"/>
+        <mass value="${rotor_mass}"/>
        <inertia
-        ixx="1e-6"
-        ixy="0"
-        ixz="0"
-        iyy="1e-6"
-        iyz="0"
-        izz="0.0003716"/>
+          ixx="0.0003716"
+          ixy="0"
+          ixz="0"
+          iyy="0.0003716"
+          iyz="0"
+          izz="0.0003716"/>
       </inertial>
     </link>

File: ros2_ws/src/pendulum_control/urdf/qube_constants.xacro (robot description, xacro)
@@ -8,6 +8,6 @@
   <xacro:property name="rotor_height" value="0.0104"/>
   <xacro:property name="rotor_mass" value="0.095"/>
-  <xacro:property name="rotor_friction" value="0"/>
-  <xacro:property name="rotor_damping" value="0.0001"/>
+  <xacro:property name="rotor_friction" value="0.0"/>
+  <xacro:property name="rotor_damping" value="3.611e-5"/>
   <xacro:property name="pendulum_radius" value="0.0048"/>
   <xacro:property name="pendulum_length" value="0.129"/>
@@ -16,4 +16,4 @@
   <xacro:property name="pendulum_mass" value="0.024"/>
   <xacro:property name="pendulum_friction" value="0"/>
-  <xacro:property name="pendulum_damping" value="0.0001"/>
+  <xacro:property name="pendulum_damping" value="6.33e-6"/>
 </xacro:constants>
